File: TympanEarPIeceShield/Tympan_EarPiece_Shield.kicad_pcb (KiCad board)
At the start: 4 copper layers, 38 x 40 mm, 49 parts, among them J1 Tympan_SJ-3523-SMT-TR, J2 Tympan_SJ-3524-SMT-TR-PI, J3 USB_B_Mini, J4 USB_B_Mini, J5 Conn_01x01, J6 Conn_01x01, P1 CONN_01X06, P2 CONN_01X06, P3 CONN_01X06, P4 CONN_01X06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

Commit message: Tidy silk
Parts:
- moved G*** 3.30 mm to (133.8, 76.2)
- moved G*** 1.20 mm to (133.8, 61.8)
Other:
- board text added: "Tympan BTE Shield"
- board text added: "www.tympan.org"
- board text removed: "Tympan EarPiece Shield"
- board text removed: "www.tympan.org github.com/tympan"
Changed lines of the file:
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@@
     (38 B.Mask user)
     (39 F.Mask user)
-    (40 Dwgs.User user)
+    (40 Dwgs.User user hide)
     (41 Cmts.User user hide)
     (42 Eco1.User user hide)
@@
   )
   (setup
-    (last_trace_width 0.2032)
+    (last_trace_width 0.25)
     (user_trace_width 0.1778)
     (user_trace_width 0.2032)
@@
   )
   (module Graphics:Tympan_LOGO (layer B.Cu)
-    (at 133.85 60.58 180)
+    (at 133.85 61.78 180)
     (attr smd)
     (fp_text reference G*** (at 0 0 180) (layer B.SilkS) hide
@@
   )
   (module Graphics:oshwa-logo-gear (layer B.Cu)
-    (at 133.85 79.48 180)
+    (at 133.85 76.18 180)
     (attr smd)
     (fp_text reference G*** (at 0 0 180) (layer B.SilkS) hide
@@
     (effects (font (size 0.762 0.762) (thickness 0.1778)))
   )
-  (gr_text "Tympan\nEarPiece Shield" (at 129.15 84.18) (layer F.SilkS)
-    (effects (font (size 1.25 1.25) (thickness 0.25)) (justify left))
-  )
-  (gr_text INPUT (at 118.15 60.48) (layer B.SilkS)
+  (gr_text "Tympan BTE Shield" (at 124.85 84.98) (layer F.SilkS)
+    (effects (font (size 1.25 1.2) (thickness 0.25)) (justify left))
+  )
+  (gr_text INPUT (at 121.95 64.38) (layer B.SilkS)
     (effects (font (size 1 1) (thickness 0.2)) (justify mirror))
   )
-  (gr_text OUTPUT (at 148.9 60.48) (layer B.SilkS)
+  (gr_text OUTPUT (at 146.15 64.48) (layer B.SilkS)
     (effects (font (size 1 1) (thickness 0.2)) (justify mirror))
   )
@@
   (gr_arc (start 116.6 84.73) (end 114.85 84.605) (angle -95.72216304) (layer Edge.Cuts) (width 0.2))
   (gr_line (start 116.650106 86.483743) (end 151.1 86.48) (angle 90) (layer Edge.Cuts) (width 0.15))
-  (gr_text "www.tympan.org\ngithub.com/tympan" (at 133.85 71.98) (layer B.SilkS)
+  (gr_text www.tympan.org (at 133.85 83.18) (layer B.SilkS)
     (effects (font (size 1 1) (thickness 0.2)) (justify mirror))
   )
-  (gr_text "Designed in Brooklyn, NY USA" (at 133.775 53.98) (layer B.SilkS)
+  (gr_text "Designed in Brooklyn, NY USA" (at 133.85 54.48) (layer B.SilkS)
     (effects (font (size 1 1) (thickness 0.2)) (justify mirror))
   )
@@
   (gr_line (start 151.1 46.48) (end 116.650536 46.479993) (angle 90) (layer Edge.Cuts) (width 0.15))
   (gr_line (start 152.85 84.73) (end 152.85 48.23) (angle 90) (layer Edge.Cuts) (width 0.15))
-  (gr_text "TYMPAN EARPIECE SHIELD" (at 133.85 68.48) (layer B.SilkS)
+  (gr_text "TYMPAN EARPIECE SHIELD" (at 133.85 69.28) (layer B.SilkS)
     (effects (font (size 1.524 1.524) (thickness 0.25)) (justify mirror))
   )
